Commit message: Convert zed-yolo-ros from submodule to regular directory

File: p3dx_description/urdf/materials.xacro (robot description, xacro)
@@ -35,3 +35,6 @@
 		<color rgba="0.038 0.038 0.038 1.0"/>
 	</material>
+	<material name="swivel">
+  		<color rgba="0.5 0.5 0.5 1"/>
+	</material>
 </robot>

File: p3dx_description/urdf/pioneer3dx.xacro (robot description, xacro)
@@ -37,4 +37,7 @@
 		<color rgba="0.038 0.038 0.038 1.0"/>
 	</material>
+	<material name="swivel">
+  		<color rgba="0.5 0.5 0.5 1"/>
+	</material>
 	<!-- chassis -->
 	<link name="base_link">
