Commit message: Recovered changes after broken ref issue

File: p3dx_description/urdf/pioneer3dx.urdf (robot description, URDF)
Before this commit: robot pioneer3dx, 13 links, 12 joints
Links:
- added link zed2i_baro_link
- added link zed2i_base_link
- added link zed2i_camera_center; collision mesh filename=package://p3dx_description/urdf/zed/meshes/zed2i.stl; visual mesh filename=package://p3dx_description/urdf/zed/meshes/zed2i.stl
- added link zed2i_left_camera_frame
- added link zed2i_left_camera_optical_frame
- added link zed2i_mag_link
- added link zed2i_right_camera_frame
- added link zed2i_right_camera_optical_frame
- added link zed2i_temp_left_link
- added link zed2i_temp_right_link
Joints:
- added joint zed2i_baro_joint: type fixed, parent zed2i_camera_center, child zed2i_baro_link, origin xyz=0 0 0 rpy=0 0 0
- added joint zed2i_base_joint: type fixed, parent base_link, child zed2i_base_link, origin xyz=0.05 0.0 1.094 rpy=0.0 0.0 0.0
- added joint zed2i_camera_center_joint: type fixed, parent zed2i_base_link, child zed2i_camera_center, origin xyz=0 0 0.015 rpy=0 0.0 0
- added joint zed2i_left_camera_joint: type fixed, parent zed2i_camera_center, child zed2i_left_camera_frame, origin xyz=0 0.06 0 rpy=0 0 0
- added joint zed2i_left_camera_optical_joint: type fixed, parent zed2i_left_camera_frame, child zed2i_left_camera_optical_frame, origin xyz=-0.01 0 0 rpy=-1.5707963267948966 0.0 -1.5707963267948966
- added joint zed2i_mag_joint: type fixed, parent zed2i_camera_center, child zed2i_mag_link, origin xyz=0 0 0 rpy=0 0 0
- added joint zed2i_right_camera_joint: type fixed, parent zed2i_camera_center, child zed2i_right_camera_frame, origin xyz=0 -0.06 0 rpy=0 0 0
- added joint zed2i_right_camera_optical_joint: type fixed, parent zed2i_right_camera_frame, child zed2i_right_camera_optical_frame, origin xyz=-0.01 0 0 rpy=-1.5707963267948966 0.0 -1.5707963267948966
- added joint zed2i_temp_left_joint: type fixed, parent zed2i_left_camera_frame, child zed2i_temp_left_link, origin xyz=0 0 0 rpy=0 0 0
- added joint zed2i_temp_right_joint: type fixed, parent zed2i_right_camera_frame, child zed2i_temp_right_link, origin xyz=0 0 0 rpy=0 0 0

File: p3dx_description/urdf/pioneer3dx.xacro (robot description, xacro)
@@ -22,4 +22,5 @@
 	<!-- import the pioneer 3dx's wheels -->
 	<xacro:include filename="$(find p3dx_description)/urdf/pioneer3dx_wheel.xacro" />
+	<xacro:include filename="$(find p3dx_description)/urdf/zed/zed_macro.urdf.xacro" />
 	<material name="SonarYellow">
 		<color rgba="0.715 0.583 0.210 1.0"/>
@@ -36,4 +37,7 @@
 	<material name="TopBlack">
 		<color rgba="0.038 0.038 0.038 1.0"/>
+	</material>
+	<material name="swivel">
+  		<color rgba="0.5 0.5 0.5 1"/>
 	</material>
 	<!-- chassis -->
@@ -285,3 +289,6 @@
 		<child link="upper_top_plate" />
 	</joint>
+	<xacro:zed_camera name="zed2i" model="zed2i" parent="base_link">
+		<origin xyz="0.05 0.0 1.094" rpy="0.0 0.0 0.0"/>
+	</xacro:zed_camera>
 </robot>

Commit message: Edits to xacro file transformations

File: p3dx_description/urdf/pioneer3dx.urdf (robot description, URDF)
Before this commit: robot pioneer3dx, 23 links, 22 joints
Joints:
- joint zed2i_base_joint: origin xyz=0.05 0.0 1.094 rpy=0.0 0.0 0.0 -> xyz=0.05 0.0 1.064 rpy=0.0 0.0 0.0

File: p3dx_description/urdf/pioneer3dx.xacro (robot description, xacro)
@@ -290,5 +290,5 @@
 	</joint>
 	<xacro:zed_camera name="zed2i" model="zed2i" parent="base_link">
-		<origin xyz="0.05 0.0 1.094" rpy="0.0 0.0 0.0"/>
+		<origin xyz="0.05 0.0 1.064" rpy="0.0 0.0 0.0"/>
 	</xacro:zed_camera>
 </robot>
